Commit message: feat: change robot colours

File: catkin_ws/src/my_robot/urdf/my_robot.xacro (robot description, xacro)
@@ -160,11 +160,11 @@
   </joint>
   <gazebo reference="chassis">
-    <material>Gazebo/White</material>
+    <material>Gazebo/Red</material>
   </gazebo>
   <gazebo reference="left_wheel">
-    <material>Gazebo/Black</material>
+    <material>Gazebo/Green</material>
   </gazebo>
   <gazebo reference="right_wheel">
-    <material>Gazebo/Black</material>
+    <material>Gazebo/Green</material>
   </gazebo>
 </robot>
